Commit message: Minor debugging changes

File: resources/robots/b1z1_current/urdf/b1z1_genesis.urdf (robot description, URDF)
Before this commit: robot b1z1_description, 29 links, 28 joints
Joints:
- joint base_static_joint: origin xyz=0.3 0 0.09 rpy=0 0 0 -> xyz=0.3 0 0.10 rpy=0 0 0

Commit message: small update to URDF to align with real robot

File: resources/robots/b1z1_current/urdf/b1z1_genesis.urdf (robot description, URDF)
Before this commit: robot b1z1_description, 29 links, 28 joints
Joints:
- joint base_static_joint: origin xyz=0.3 0 0.10 rpy=0 0 0 -> xyz=0.3 0 0.09 rpy=0 0 0
